File: hardware/silvaback/silvaback.kicad_sch (KiCad schematic)
At the start: 29 parts, among them J1 AC_IN, J2 FAN, K1 SANYOU_SRD_Form_C, SW1 RotaryEncoder_Switch, U1 SSD1306_OLED_SCREEN

Commit message: working encoder menu
Parts:
- added unit 3 of U2
- gave numbers to parts that had none: 10
Connections:
- net ENCODER_BUTTON: now also U2.5
- new net MCU_ENC_BUTTON: U2.6
Other:
- moved on the sheet: U2A, U2B, U2G
